File: hardware/esp-wifisensor.sch (EAGLE design)
At the start: 16 parts

Commit message: hardware: updated schematics and pcb
Parts:
- removed C5, C6: 100n, rcl:C-EUC1206K
- added G1: BHC-18650-1P, BHC-18650-1P:BHC-18650-1P
- C1: value 470u -> 1500u; device rcl:CPOL-EUD/7343-31W -> ED1E152MNN1225:CPOL-EUE5-13
- C2, C3: value 470u -> 100n; device rcl:CPOL-EUD/7343-31W -> rcl:C-EUC1206K
Connections:
- net GND: now also C2.2, C3.2, G1.-, JP1.4; no longer C2.-, C3.-, C5.2, C6.2, JP1.1
- net N$10: now also JP1.1; no longer JP1.2
- net N$5: now also JP1.3; no longer JP1.4
- net N$8: now also JP1.2; no longer JP1.3
- net VCC: now also C2.1, C3.1, G1.+; no longer C2.+, C3.+, C5.1, C6.1
Other:
- moved on the sheet: C1, C4, JP1
Changed lines of the file:
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@@
 <part name="U$1" library="BMP180_module" deviceset="BMP180" device=""/>
 <part name="U$2" library="SHT-21_module" deviceset="SHT-21" device=""/>
-<part name="C1" library="rcl" deviceset="CPOL-EU" device="D/7343-31W" value="470u"/>
-<part name="C2" library="rcl" deviceset="CPOL-EU" device="D/7343-31W" value="470u"/>
-<part name="C3" library="rcl" deviceset="CPOL-EU" device="D/7343-31W" value="470u"/>
+<part name="C2" library="rcl" deviceset="C-EU" device="C1206K" value="100n"/>
+<part name="C3" library="rcl" deviceset="C-EU" device="C1206K" value="100n"/>
 <part name="C4" library="rcl" deviceset="C-EU" device="C1206K" value="100n"/>
-<part name="C5" library="rcl" deviceset="C-EU" device="C1206K" value="100n"/>
-<part name="C6" library="rcl" deviceset="C-EU" device="C1206K" value="100n"/>
 <part name="P+1" library="supply1" deviceset="VCC" device=""/>
 <part name="P+2" library="supply1" deviceset="VCC" device=""/>
 <part name="GND2" library="supply1" deviceset="GND" device=""/>
-<part name="GND3" library="supply1" deviceset="GND" device=""/>
-<part name="GND4" library="supply1" deviceset="GND" device=""/>
 <part name="GND5" library="supply1" deviceset="GND" device=""/>
 <part name="GND6" library="supply1" deviceset="GND" device=""/>
@@
 <part name="R5" library="rcl" deviceset="R-EU_" device="M1206" value="10k"/>
 <part name="R6" library="rcl" deviceset="R-EU_" device="M1206" value="10k"/>
+<part name="G1" library="BHC-18650-1P" deviceset="BHC-18650-1P" device=""/>
+<part name="P+5" library="supply1" deviceset="VCC" device=""/>
+<part name="GND9" library="supply1" deviceset="GND" device=""/>
+<part name="C1" library="ED1E152MNN1225" deviceset="CPOL-EU" device="E5-13" value="1500u"/>
 </parts>
 <sheets>
@@
 <instance part="U$1" gate="G$1" x="109.22" y="71.12" rot="MR0"/>
 <instance part="U$2" gate="G$1" x="109.22" y="48.26" rot="MR0"/>
-<instance part="C1" gate="G$1" x="-10.16" y="50.8"/>
-<instance part="C2" gate="G$1" x="-2.54" y="50.8"/>
-<instance part="C3" gate="G$1" x="5.08" y="50.8"/>
-<instance part="C4" gate="G$1" x="12.7" y="50.8"/>
-<instance part="C5" gate="G$1" x="86.36" y="17.78"/>
-<instance part="C6" gate="G$1" x="93.98" y="17.78"/>
-<instance part="P+1" gate="VCC" x="-10.16" y="66.04"/>
+<instance part="C2" gate="G$1" x="12.7" y="50.8"/>
+<instance part="C3" gate="G$1" x="86.36" y="17.78"/>
+<instance part="C4" gate="G$1" x="93.98" y="17.78"/>
+<instance part="P+1" gate="VCC" x="5.08" y="66.04"/>
 <instance part="P+2" gate="VCC" x="104.14" y="99.06"/>
-<instance part="GND2" gate="1" x="-10.16" y="40.64"/>
-<instance part="GND3" gate="1" x="-2.54" y="40.64"/>
-<instance part="GND4" gate="1" x="5.08" y="40.64"/>
+<instance part="GND2" gate="1" x="5.08" y="40.64"/>
 <instance part="GND5" gate="1" x="12.7" y="40.64"/>
 <instance part="GND6" gate="1" x="101.6" y="38.1"/>
@@
 <instance part="R2" gate="G$1" x="68.58" y="50.8" rot="R270"/>
 <instance part="GND10" gate="1" x="68.58" y="40.64"/>
-<instance part="JP1" gate="A" x="78.74" y="88.9" rot="MR180"/>
-<instance part="GND11" gate="1" x="73.66" y="76.2"/>
+<instance part="JP1" gate="A" x="81.28" y="86.36" rot="MR180"/>
+<instance part="GND11" gate="1" x="73.66" y="96.52" rot="R180"/>
 <instance part="R3" gate="G$1" x="91.44" y="81.28" rot="R270"/>
 <instance part="R4" gate="G$1" x="96.52" y="81.28" rot="R270"/>
 <instance part="R5" gate="G$1" x="40.64" y="91.44"/>
 <instance part="R6" gate="G$1" x="40.64" y="86.36"/>
+<instance part="G1" gate="G$1" x="-10.16" y="73.66" rot="R90"/>
+<instance part="P+5" gate="VCC" x="-10.16" y="83.82"/>
+<instance part="GND9" gate="1" x="-10.16" y="63.5"/>
+<instance part="C1" gate="G$1" x="5.08" y="50.8"/>
 </instances>
 <busses>
@@
 <segment>
 <pinref part="GND2" gate="1" pin="GND"/>
+<wire x1="5.08" y1="43.18" x2="5.08" y2="45.72" width="0.1524" layer="91"/>
 <pinref part="C1" gate="G$1" pin="-"/>
-<wire x1="-10.16" y1="43.18" x2="-10.16" y2="45.72" width="0.1524" layer="91"/>
-</segment>
-<segment>
-<pinref part="GND3" gate="1" pin="GND"/>
-<pinref part="C2" gate="G$1" pin="-"/>
-<wire x1="-2.54" y1="43.18" x2="-2.54" y2="45.72" width="0.1524" layer="91"/>
-</segment>
-<segment>
-<pinref part="GND4" gate="1" pin="GND"/>
-<pinref part="C3" gate="G$1" pin="-"/>
-<wire x1="5.08" y1="43.18" x2="5.08" y2="45.72" width="0.1524" layer="91"/>
 </segment>
 <segment>
 <pinref part="GND5" gate="1" pin="GND"/>
-<pinref part="C4" gate="G$1" pin="2"/>
+<pinref part="C2" gate="G$1" pin="2"/>
 <wire x1="12.7" y1="43.18" x2="12.7" y2="45.72" width="0.1524" layer="91"/>
 </segment>
@@
 <segment>
 <pinref part="GND7" gate="1" pin="GND"/>
-<pinref part="C5" gate="G$1" pin="2"/>
+<pinref part="C3" gate="G$1" pin="2"/>
 <wire x1="86.36" y1="10.16" x2="86.36" y2="12.7" width="0.1524" layer="91"/>
 </segment>
 <segment>
 <pinref part="GND8" gate="1" pin="GND"/>
-<pinref part="C6" gate="G$1" pin="2"/>
+<pinref part="C4" gate="G$1" pin="2"/>
 <wire x1="93.98" y1="10.16" x2="93.98" y2="12.7" width="0.1524" layer="91"/>
 </segment>
@@
 </segment>
 <segment>
+<pinref part="GND9" gate="1" pin="GND"/>
+<pinref part="G1" gate="G$1" pin="-"/>
+<wire x1="-10.16" y1="66.04" x2="-10.16" y2="68.58" width="0.1524" layer="91"/>
+</segment>
+<segment>
+<pinref part="JP1" gate="A" pin="4"/>
 <pinref part="GND11" gate="1" pin="GND"/>
-<pinref part="JP1" gate="A" pin="1"/>
-<wire x1="76.2" y1="83.82" x2="73.66" y2="83.82" width="0.1524" layer="91"/>
-<wire x1="73.66" y1="83.82" x2="73.66" y2="78.74" width="0.1524" layer="91"/>
+<wire x1="78.74" y1="88.9" x2="73.66" y2="88.9" width="0.1524" layer="91"/>
+<wire x1="73.66" y1="88.9" x2="73.66" y2="93.98" width="0.1524" layer="91"/>
 </segment>
 </net>
@@
 <wire x1="25.4" y1="58.42" x2="12.7" y2="58.42" width="0.1524" layer="91"/>
 <wire x1="12.7" y1="58.42" x2="5.08" y2="58.42" width="0.1524" layer="91"/>
-<wire x1="5.08" y1="58.42" x2="-2.54" y2="58.42" width="0.1524" layer="91"/>
-<wire x1="-10.16" y1="58.42" x2="-10.16" y2="63.5" width="0.1524" layer="91"/>
-<pinref part="C1" gate="G$1" pin="+"/>
-<wire x1="-10.16" y1="53.34" x2="-10.16" y2="58.42" width="0.1524" layer="91"/>
-<pinref part="C2" gate="G$1" pin="+"/>
-<wire x1="-10.16" y1="58.42" x2="-2.54" y2="58.42" width="0.1524" layer="91"/>
-<wire x1="-2.54" y1="58.42" x2="-2.54" y2="53.34" width="0.1524" layer="91"/>
-<pinref part="C3" gate="G$1" pin="+"/>
+<wire x1="5.08" y1="58.42" x2="5.08" y2="63.5" width="0.1524" layer="91"/>
 <wire x1="5.08" y1="53.34" x2="5.08" y2="58.42" width="0.1524" layer="91"/>
-<pinref part="C4" gate="G$1" pin="1"/>
+<pinref part="C2" gate="G$1" pin="1"/>
 <wire x1="12.7" y1="53.34" x2="12.7" y2="58.42" width="0.1524" layer="91"/>
-<junction x="-10.16" y="58.42"/>
-<junction x="-2.54" y="58.42"/>
 <junction x="5.08" y="58.42"/>
 <junction x="12.7" y="58.42"/>
+<pinref part="C1" gate="G$1" pin="+"/>
 </segment>
 <segment>
@@
 </segment>
 <segment>
-<pinref part="C6" gate="G$1" pin="1"/>
+<pinref part="C4" gate="G$1" pin="1"/>
 <wire x1="93.98" y1="20.32" x2="93.98" y2="22.86" width="0.1524" layer="91"/>
 <wire x1="93.98" y1="22.86" x2="86.36" y2="22.86" width="0.1524" layer="91"/>
-<pinref part="C5" gate="G$1" pin="1"/>
+<pinref part="C3" gate="G$1" pin="1"/>
 <wire x1="86.36" y1="22.86" x2="86.36" y2="20.32" width="0.1524" layer="91"/>
 <pinref part="P+3" gate="VCC" pin="VCC"/>
@@
 <junction x="15.24" y="86.36"/>
 </segment>
+<segment>
+<pinref part="G1" gate="G$1" pin="+"/>
+<pinref part="P+5" gate="VCC" pin="VCC"/>
+<wire x1="-10.16" y1="78.74" x2="-10.16" y2="81.28" width="0.1524" layer="91"/>
+</segment>
 </net>
 <net name="N$2" class="0">
@@
 <pinref part="U1" gate="G$1" pin="GPIO0"/>
 <wire x1="58.42" y1="66.04" x2="68.58" y2="66.04" width="0.1524" layer="91"/>
-<wire x1="68.58" y1="66.04" x2="68.58" y2="91.44" width="0.1524" layer="91"/>
-<pinref part="JP1" gate="A" pin="4"/>
-<wire x1="68.58" y1="91.44" x2="76.2" y2="91.44" width="0.1524" layer="91"/>
+<wire x1="68.58" y1="66.04" x2="68.58" y2="86.36" width="0.1524" layer="91"/>
 <pinref part="R5" gate="G$1" pin="2"/>
+<wire x1="68.58" y1="86.36" x2="68.58" y2="91.44" width="0.1524" layer="91"/>
 <wire x1="68.58" y1="91.44" x2="45.72" y2="91.44" width="0.1524" layer="91"/>
-<junction x="68.58" y="91.44"/>
+<pinref part="JP1" gate="A" pin="3"/>
+<wire x1="78.74" y1="86.36" x2="68.58" y2="86.36" width="0.1524" layer="91"/>
+<junction x="68.58" y="86.36"/>
 </segment>
 </net>
@@
 <pinref part="U1" gate="G$1" pin="TX"/>
 <wire x1="58.42" y1="76.2" x2="63.5" y2="76.2" width="0.1524" layer="91"/>
-<wire x1="63.5" y1="76.2" x2="63.5" y2="88.9" width="0.1524" layer="91"/>
-<pinref part="JP1" gate="A" pin="3"/>
-<wire x1="76.2" y1="88.9" x2="63.5" y2="88.9" width="0.1524" layer="91"/>
+<wire x1="63.5" y1="76.2" x2="63.5" y2="83.82" width="0.1524" layer="91"/>
+<pinref part="JP1" gate="A" pin="2"/>
+<wire x1="78.74" y1="83.82" x2="63.5" y2="83.82" width="0.1524" layer="91"/>
 </segment>
 </net>
@@
 <pinref part="U1" gate="G$1" pin="RX"/>
 <wire x1="58.42" y1="73.66" x2="66.04" y2="73.66" width="0.1524" layer="91"/>
-<wire x1="66.04" y1="73.66" x2="66.04" y2="86.36" width="0.1524" layer="91"/>
-<pinref part="JP1" gate="A" pin="2"/>
-<wire x1="76.2" y1="86.36" x2="66.04" y2="86.36" width="0.1524" layer="91"/>
-</segment>
-</net>
+<wire x1="66.04" y1="73.66" x2="66.04" y2="81.28" width="0.1524" layer="91"/>
+<pinref part="JP1" gate="A" pin="1"/>
+<wire x1="78.74" y1="81.28" x2="66.04" y2="81.28" width="0.1524" layer="91"/>
+</segment>
+</net>
